File: PCB/rev0/arduino_pcb/arduino_pcb.sch (KiCad schematic (older format))
At the start: 8 parts

Commit message: PCB_rev0
Parts:
- added J5: LED1, Connector_Molex:Molex_SPOX_5267-04A_1x04_P2.50mm_Vertical, symbol Connector:Conn_01x04_Male
- added J6: OPERATE, Connector_Molex:Molex_SPOX_5267-02A_1x02_P2.50mm_Vertical, symbol Connector:Conn_01x02_Male
- added J7: STATE, Connector_Molex:Molex_SPOX_5267-02A_1x02_P2.50mm_Vertical, symbol Connector:Conn_01x02_Male
- added J8: FREQ, Connector_Molex:Molex_SPOX_5267-02A_1x02_P2.50mm_Vertical, symbol Connector:Conn_01x02_Male
- added J9: LED2, Connector_Molex:Molex_SPOX_5267-04A_1x04_P2.50mm_Vertical, symbol Connector:Conn_01x04_Male
- added R1, R2, R3: 4.7K, Resistor_THT:R_Axial_DIN0207_L6.3mm_D2.5mm_P10.16mm_Horizontal, symbol Device:R
- added SW1: OPERATE, Button_Switch_THT:SW_PUSH-12mm, symbol Switch:SW_Push
- added SW2: STATE, Button_Switch_THT:SW_PUSH-12mm, symbol Switch:SW_Push
- added SW3: FREQ, Button_Switch_THT:SW_PUSH-12mm, symbol Switch:SW_Push
- J1: renamed from J?; footprint (none) -> PJ-076:CUI_PJ-076
- J2: renamed from J?; value Conn_Coaxial -> TDT0; footprint (none) -> Connector_Coaxial:BNC_Amphenol_B6252HB-NPP3G-50_Horizontal
- J3: renamed from J?; value Conn_Coaxial -> TDT1; footprint (none) -> Connector_Coaxial:BNC_Amphenol_B6252HB-NPP3G-50_Horizontal
- J4: renamed from J?; value Conn_Coaxial -> TDT2; footprint (none) -> Connector_Coaxial:BNC_Amphenol_B6252HB-NPP3G-50_Horizontal
- gave numbers to parts that had none: 4
Connections:
- net +12V: now also J5.1 (Pin_1), J9.1 (Pin_1)
- net +3V3: now also J6.1 (Pin_1), J7.1 (Pin_1), J8.1 (Pin_1), SW1.2, SW2.2, SW3.2
- net BLUELED: now also J5.4 (Pin_4), J9.4 (Pin_4)
- net GND: now also A1.29 (GND), A1.4 (GND), Q2.3 (S), R1.2, R2.2, R3.2
- net GREENLED: now also J5.2 (Pin_2), J9.2 (Pin_2)
- net OPERATE: now also J6.2 (Pin_2), R2.1, SW1.1
- net REDLED: now also J5.3 (Pin_3), J9.3 (Pin_3)
- net STATE: now also J7.2 (Pin_2), R3.1, SW2.1
- net FREQ: now reaches A1.11 (D8)
- net FREQ: now also J8.2 (Pin_2), R1.1, SW3.1
- no-connect marks 17 -> 16
Other:
- moved on the sheet: A1, J1, J2, J3, J4, Q1, Q2, Q3
