File: PCB/rev0/arduino_pcb/arduino_pcb.kicad_pcb (KiCad board)
At the start: 2 copper layers, 126 x 70 mm, 23 parts, among them J1 Jack-DC, J2 TDT0, J3 TDT1, J4 TDT2, J5 LED1, J6 OPERATE, J7 STATE, J8 FREQ, J9 LED2, Q1 IRF510PBF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

Commit message: PCB_gerber update
Other:
- board text added: "FREQ"
- board text added: "LED1 VGRB"
- board text added: "LED2 VGRB"
- board text added: "OPERATE"
- board text added: "STATE"
- board text added: "TDT0"
- board text added: "TDT1"
- board text added: "TDT2"
