File: PCB/electrode_FPCB/electrode_FPCB_rev0/electrode_FPCB_rev1.2d.kicad_pcb (KiCad board)
At the start: 2 copper layers, 68 x 67.5 mm, 8 parts

Commit message: vr electrode pad v1.2d (fix silkscreen)
Other:
- board text added: "VR EEG electrode v1.2d SJLEE/JGSHIN"
- board text removed: "VR EEG electrode v1.2c"
Changed lines of the file:
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@@
       (drillshape 0)
       (scaleselection 1)
-      (outputdirectory "rev1.2c_gerber/"))
+      (outputdirectory "rev1.2d_gerber/"))
   )
   (net 0 "")
@@
   (gr_arc (start 125.3 55.7) (end 121.800001 59.299999) (angle -269.1930705) (layer Edge.Cuts) (width 0.1))
   (gr_arc (start 67.3 55.7) (end 70.799999 52.100001) (angle -269.1930705) (layer Edge.Cuts) (width 0.1))
-  (gr_text "VR EEG electrode v1.2c\n" (at 96.25 77.25 90) (layer F.SilkS)
+  (gr_text "VR EEG electrode v1.2d\nSJLEE/JGSHIN" (at 96.25 77.25 90) (layer F.SilkS)
     (effects (font (size 1 1) (thickness 0.15)))
   )

Commit message: minor changes
Other:
- board text added: "Back adhesive, 3M Tape"
- board text added: "Reinforcing plate"
